File: Hardware/GLCD_Adapter.brd (EAGLE design)
At the start: 160 x 100 mm, 17 parts, among them IC2 74AC245N, IC3 74AC245N, J1 22-27-2031-03, J2 22-05-7068-06, X3 STM32F4_DISC

Commit message: - removed USB Mounted Sem - Filehandler prepared for MP3Player
Change-Id: Ie52e104650d60b68fc964640fa024eed4f39e2ff
Parts:
- removed J1: 22-27-2031-03, con-molex:6410-03
- removed J2: 22-05-7068-06, con-molex:7395-06
- removed JP1: (no value), pinhead:1X20
- removed JP3: (no value), pinhead:1X07
- added C10, C11, C12: 100µ, rcl:E2-5
- added C5: 10µ, rcl:E2-5
- added C6, C9: 4µ7, rcl:E2-5
- added C7, C8: 100n, rcl:C1206
- added IC1: 78L05, v-reg:78XXL
- added Q1, Q4, Q6, Q8: BSS123, transistor-small-signal:SOT23
- added Q2, Q5, Q7, Q9: SI4427DY, transistor-power:SO-08
- added Q3: SI4466DY, transistor-power:SO-08
- added R10, R11, R12, R3, R5, R6, R7, R9: 1k, rcl:R1206
- added R4: 10R, rcl:0414/15
- added R8: (no value), rcl:R1206
- added X1: PWR, con-ptr500:AK500/3
- added X10: PD89, con-molex:22-23-2031
- added X2: 22-23-2031, con-molex:22-23-2031
- added X4: OUT1, con-ptr500:AK500/2
- added X5: 22-23-2021, con-molex:22-23-2021
- added X6: OUT2, con-ptr500:AK500/2
- added X7: PD1415, con-molex:22-23-2031
- added X8: PD1213, con-molex:22-23-2031
- added X9: PD1011, con-molex:22-23-2031
- moved SJ2 207.0 mm to (-41.9, 77.5)
- moved JP2 196.6 mm to (-27.9, 74.9)
- moved H1 188.4 mm to (20.3, 52.1), flipped to the bottom, turned to 180 degrees
- moved SJ1 172.5 mm to (-40.6, 47.0)
- moved IC3 160.4 mm to (85.1, 26.7)
- moved C1 148.4 mm to (16.5, -20.3)
- moved C3 148.4 mm to (16.5, -41.9)
- moved C4 148.4 mm to (16.5, -48.3)
- moved R2 148.4 mm to (16.5, -35.6)
- moved C2 148.4 mm to (16.5, -25.4)
- moved R1 148.4 mm to (16.5, -30.5)
- moved X3 119.4 mm to (68.6, 36.8), turned to 90 degrees
- moved IC2 114.1 mm to (55.9, 26.7)
Connections:
- removed net A: JP2.3
- removed net K: JP2.1
- removed net NC: JP1.20
- removed net SD_CD: JP3.1
- removed net SD_CS: JP3.7
- removed net SD_D0: JP3.2
- removed net SD_DI: JP3.6
- removed net SD_SCK: JP3.4
- removed net V0: JP1.3
- removed net VCC: C1.1, C2.1, C3.1, C4.1, IC2.1, IC2.20, IC3.20, JP3.5, SJ1.1, SJ2.1, X3.R3, X3.R4
- removed net VEE: JP1.17
- removed net VSS: JP1.1
- new net +12V: C12.+, C6.+, C7.1, IC1.IN, Q2.1, Q2.2, Q2.3, Q5.1, Q5.2, Q5.3, X1.2
- new net +24V: C10.+, C11.+, C5.+, Q7.1, Q7.2, Q7.3, Q9.1, Q9.2, Q9.3, X1.3
- new net +5V: C1.1, C2.1, C3.1, C4.1, C8.1, C9.+, H1.16, H1.2, IC1.OUT, IC2.1, IC2.20, IC3.20, SJ1.1, SJ2.1, X3.R3, X3.R4
- new net ENC_A: X2.1, X3.R25
- new net ENC_B: X2.3, X3.R26
- new net ENC_UB: X3.R24, X5.1
- new net IN_BL: R5.1, X3.L11
- new net IN_BUZZ: R6.1, X3.L14
- new net IN_LED: R8.1, X3.L13
- new net IN_OUT1: R12.1, X3.L16
- new net IN_OUT2: R10.1, X3.R43
- new net LED1: Q7.5, Q7.6, Q7.7, Q7.8, X6.2
- new net LED2: Q9.5, Q9.6, Q9.7, Q9.8, X4.2
- new net N$10: Q7.4, R9.2
- new net N$11: Q4.1, R8.2
- new net N$12: Q6.3, R9.1
- new net N$13: Q6.1, R10.2
- new net N$14: Q9.4, R11.2
- new net N$15: Q8.3, R11.1
- new net N$16: Q8.1, R12.2
- new net N$20: X10.2, X3.L40
- new net N$21: X10.1, X3.L41
- new net N$22: X3.L42, X9.2
- new net N$23: X3.L43, X9.1
- new net N$24: X3.L44, X8.2
- new net N$25: X3.L45, X8.1
- new net N$26: X3.L46, X7.2
- new net N$27: X3.L47, X7.1
- new net N$3: Q2.4, R3.2
- new net N$4: Q1.3, R3.1
- new net N$5: Q2.5, Q2.6, Q2.7, Q2.8, R4.1
- new net N$6: Q1.1, R5.2
- new net N$7: Q5.4, R7.2
- new net N$8: Q3.4, R6.2
- new net N$9: Q4.3, R7.1
- net !CE: no longer JP1.15
- net !RD: no longer JP1.5
- net !RST: no longer JP1.16
- net !WR: no longer JP1.6
- net BL: now also JP2.3, R4.2
- net BUZZ: now also Q3.5, Q3.6, Q3.7, Q3.8
- net C/D: no longer JP1.4
- net D0: no longer JP1.7
- net D1: no longer JP1.8
- net D2: no longer JP1.9
- net D3: no longer JP1.10
- net D4: no longer JP1.11
- net D5: no longer JP1.12
- net D6: no longer JP1.13
- net D7: no longer JP1.14
- net FS1: no longer JP1.19
- net GND: now also C10.-, C11.-, C12.-, C5.-, C6.-, C7.2, C8.2, C9.-, IC1.GND, JP2.1, Q1.2, Q3.1, Q3.2, Q3.3, Q4.2, Q6.2, Q8.2, X1.1, X10.3, X2.2, X4.1, X5.2, X6.1, X7.3, X8.3, X9.3; no longer JP3.3
- net IN_!CE: now also X3.L38
- net IN_!RD: now also X3.L35
- net IN_!RST: now also X3.L37
- net IN_!WR: now also X3.L36
- net IN_A0: now also X3.L22
- net IN_A1: now also X3.L21
- net IN_A2: now also X3.L24
- net IN_C/D: now also X3.L39
- net IN_D0: now also X3.L26
- net IN_D1: now also X3.L27
- net IN_D2: now also X3.L28
- net IN_D3: now also X3.L29
- net IN_D4: now also X3.L30
- net IN_D5: now also X3.L31
- net IN_D6: now also X3.L32
- net IN_D7: now also X3.L33
- net LED: now also Q5.5, Q5.6, Q5.7, Q5.8
- net MD2: no longer JP1.18
- net VDD: no longer H1.16, H1.2, JP1.2
Routing:
- net GND: track 0.00 -> 1008.3 mm, vias 0 -> 9
- net +12V: track 0.00 -> 417.7 mm, vias 0 -> 2
- net +24V: track 0.00 -> 405.1 mm
- net +5V: track 0.00 -> 397.2 mm, vias 0 -> 6
- net N$14: track 0.00 -> 205.6 mm
- net N$10: track 0.00 -> 185.4 mm
- net N$8: track 0.00 -> 180.4 mm
- net N$2: track 0.00 -> 174.7 mm
- net IN_!RST: track 0.00 -> 169.9 mm, vias 0 -> 4
- net !RD: track 0.00 -> 157.5 mm, vias 0 -> 4
- net N$3: track 0.00 -> 146.5 mm
- net IN_D7: track 0.00 -> 117.3 mm
- net N$1: track 0.00 -> 105.6 mm, vias 0 -> 2
- net IN_D3: track 0.00 -> 98.2 mm, vias 0 -> 2
- net IN_D1: track 0.00 -> 97.4 mm, vias 0 -> 2
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Other:
- board size 160 x 100 mm -> 148.6 x 108.9 mm
