File: Hardware/GLCD_Adapter.sch (EAGLE design)
At the start: 17 parts, among them IC2 74AC245N, IC3 74AC245N, J1 22-27-2031-03, J2 22-05-7068-06, X3 STM32F4_DISC

Commit message: - removed USB Mounted Sem - Filehandler prepared for MP3Player
Change-Id: Ie52e104650d60b68fc964640fa024eed4f39e2ff
Parts:
- removed J1: 22-27-2031-03, con-molex:22-27-2031-03
- removed J2: 22-05-7068-06, con-molex:22-05-7068-06
- removed JP1: (no value), pinhead:PINHD-1X20
- removed JP3: (no value), pinhead:PINHD-1X7
- added C10, C11, C12: 100µ, rcl:CPOL-EUE2-5
- added C5: 10µ, rcl:CPOL-EUE2-5
- added C6, C9: 4µ7, rcl:CPOL-EUE2-5
- added C7, C8: 100n, rcl:C-EUC1206
- added IC1: 78L05, v-reg:78XXL
- added Q1, Q4, Q6, Q8: BSS123, transistor-small-signal:BSS123
- added Q2, Q5, Q7, Q9: SI4427DY, transistor-power:P-MOSFET-SO8
- added Q3: SI4466DY, transistor-power:N-MOSFET-SO8S
- added R10, R11, R12, R3, R5, R6, R7, R9: 1k, rcl:R-EU_R1206
- added R4: 10R, rcl:R-EU_0414/15
- added R8: (no value), rcl:R-EU_R1206
- added X1: PWR, con-ptr500:AK500/3
- added X10: PD89, con-molex:22-23-2031
- added X2: 22-23-2031, con-molex:22-23-2031
- added X4: OUT1, con-ptr500:AK500/2
- added X5: 22-23-2021, con-molex:22-23-2021
- added X6: OUT2, con-ptr500:AK500/2
- added X7: PD1415, con-molex:22-23-2031
- added X8: PD1213, con-molex:22-23-2031
- added X9: PD1011, con-molex:22-23-2031
Connections:
- removed net A: JP2.3
- removed net K: JP2.1
- removed net NC: JP1.20
- removed net SD_CD: JP3.1
- removed net SD_CS: JP3.7
- removed net SD_D0: JP3.2
- removed net SD_DI: JP3.6
- removed net SD_SCK: JP3.4
- removed net V0: JP1.3
- removed net VCC: C1.1, C2.1, C3.1, C4.1, IC2A.DIR, IC2P.VCC, IC3P.VCC, JP3.5, SJ1.1, SJ2.1, X3PWR.5V@1, X3PWR.5V@2
- removed net VDD: H1.VCC, JP1.2
- removed net VEE: JP1.17
- removed net VSS: JP1.1
- new net +12V: C12.+, C6.+, C7.1, IC1.IN, Q2.S, Q5.S, X1-2.KL
- new net +24V: C10.+, C11.+, C5.+, Q7.S, Q9.S, X1-3.KL
- new net +5V: C1.1, C2.1, C3.1, C4.1, C8.1, C9.+, H1.VCC, IC1.OUT, IC2A.DIR, IC2P.VCC, IC3P.VCC, SJ1.1, SJ2.1, X3PWR.5V@1, X3PWR.5V@2
- new net ENC_A: X2-1.S, X3PORTB.PB4
- new net ENC_B: X2-3.S, X3PORTB.PB5
- new net ENC_UB: X3PORTB.PB7, X5-1.S
- new net IN_BL: R5.1, X3PORTA.PA1
- new net IN_BUZZ: R6.1, X3PORTA.PA2
- new net IN_LED: R8.1, X3PORTA.PA3
- new net IN_OUT1: R12.1, X3PORTA.PA4
- new net IN_OUT2: R10.1, X3PORTA.PA8
- new net LED1: Q7.D, X6-2.KL
- new net LED2: Q9.D, X4-2.KL
- new net N$10: Q7.G, R9.2
- new net N$11: Q4.G, R8.2
- new net N$12: Q6.D, R9.1
- new net N$13: Q6.G, R10.2
- new net N$14: Q9.G, R11.2
- new net N$15: Q8.D, R11.1
- new net N$16: Q8.G, R12.2
- new net N$20: X10-2.S, X3PORTD.PD8
- new net N$21: X10-1.S, X3PORTD.PD9
- new net N$22: X3PORTD.PD10, X9-2.S
- new net N$23: X3PORTD.PD11, X9-1.S
- new net N$24: X3PORTD.PD12, X8-2.S
- new net N$25: X3PORTD.PD13, X8-1.S
- new net N$26: X3PORTD.PD14, X7-2.S
- new net N$27: X3PORTD.PD15, X7-1.S
- new net N$3: Q2.G, R3.2
- new net N$4: Q1.D, R3.1
- new net N$5: Q2.D, R4.1
- new net N$6: Q1.G, R5.2
- new net N$7: Q5.G, R7.2
- new net N$8: Q3.G, R6.2
- new net N$9: Q4.D, R7.1
- net !CE: no longer JP1.15
- net !RD: no longer JP1.5
- net !RST: no longer JP1.16
- net !WR: no longer JP1.6
- net BL: now also JP2.3, R4.2
- net BUZZ: now also Q3.D
- net C/D: no longer JP1.4
- net D0: no longer JP1.7
- net D1: no longer JP1.8
- net D2: no longer JP1.9
- net D3: no longer JP1.10
- net D4: no longer JP1.11
- net D5: no longer JP1.12
- net D6: no longer JP1.13
- net D7: no longer JP1.14
- net FS1: no longer JP1.19
- net GND: now also C10.-, C11.-, C12.-, C5.-, C6.-, C7.2, C8.2, C9.-, IC1.GND, JP2.1, Q1.S, Q3.S, Q4.S, Q6.S, Q8.S, X1-1.KL, X10-3.S, X2-2.S, X4-1.KL, X5-2.S, X6-1.KL, X7-3.S, X8-3.S, X9-3.S; no longer JP3.3
- net IN_!CE: now also X3PORTB.PB14
- net IN_!RD: now also X3PORTB.PB11
- net IN_!RST: now also X3PORTB.PB13
- net IN_!WR: now also X3PORTB.PB12
- net IN_A0: now also X3PORTB.PB0
- net IN_A1: now also X3PORTB.PB1
- net IN_A2: now also X3PORTB.PB2
- net IN_C/D: now also X3PORTB.PB15
- net IN_D0: now also X3PORTE.PE8
- net IN_D1: now also X3PORTE.PE9
- net IN_D2: now also X3PORTE.PE10
- net IN_D3: now also X3PORTE.PE11
- net IN_D4: now also X3PORTE.PE12
- net IN_D5: now also X3PORTE.PE13
- net IN_D6: now also X3PORTE.PE14
- net IN_D7: now also X3PORTE.PE15
- net LED: now also Q5.D
- net MD2: no longer JP1.18
Other:
- moved on the sheet: C1, C2, C3, C4, H1, IC2, IC2P, IC3, IC3P, JP2, R1, R2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
