File: Hardware/Touch/Touch_V5.sch (EAGLE design)
At the start: 50 parts, among them IC1 78L05, IC2 74AC245N, IC3 74AC245N, Q1 BSS123, Q2 SI4427DY, Q3 SI4466DY, Q4 BSS123, Q5 SI4427DY, Q6 BSS123, Q7 SI4427DY, Q8 BSS123, Q9 SI4427DY, X1 PWR, X10 PD89, X2 22-23-2031, X3 STM32F4_DISC, X4 OUT1, X5 22-23-2021, X6 OUT2, X7 PD1415, X8 PD1213, X9 PD1011

Commit message: Change-Id: I8ad52aa35e7ba0e6f486941214efc611bf83b7b6
Parts:
- removed C10, C11, C12: 100µ, rcl:CPOL-EUE2-5
- removed C2, C3: 100n, rcl:C-EUC1206
- removed C9: 4µ7, rcl:CPOL-EUE2-5
- removed H1: (no value), GLCD-YL240:YL_24012-70-MICROMATCH
- removed IC2, IC3: 74AC245N, 74xx-eu:74AC245N
- removed JP2: (no value), pinhead:PINHD-1X3
- removed Q1, Q4, Q6, Q8: BSS123, transistor-small-signal:BSS123
- removed Q2, Q5, Q7, Q9: SI4427DY, transistor-power:P-MOSFET-SO8
- removed Q3: SI4466DY, transistor-power:N-MOSFET-SO8S
- removed R11, R12: 1k, rcl:R-EU_R1206
- removed SJ1, SJ2: (no value), jumper:SJ2WW
- removed X1: PWR, con-ptr500:AK500/3
- removed X10: PD89, con-molex:22-23-2031
- removed X2: 22-23-2031, con-molex:22-23-2031
- removed X3: STM32F4_DISC, stm32f4_disc:STM32F4_DISC
- removed X4: OUT1, con-ptr500:AK500/2
- removed X5: 22-23-2021, con-molex:22-23-2021
- removed X6: OUT2, con-ptr500:AK500/2
- removed X7: PD1415, con-molex:22-23-2031
- removed X8: PD1213, con-molex:22-23-2031
- removed X9: PD1011, con-molex:22-23-2031
- added J1: 22-27-2021-02, con-molex:22-27-2021-02
- added J2: 22-27-2041-04, con-molex:22-27-2041-04
- added JP1: ISP, pinhead:PINHD-2X3
- added LED1: PWR, led:LED3MM
- C1: device rcl:C-EUC1206 -> rcl:C-EU050-025X075
- C4: value 100n -> 10µ; device rcl:C-EUC1206 -> rcl:CPOL-EUE2-5
- C5: value 10µ -> 47n; device rcl:CPOL-EUE2-5 -> rcl:C-EU050-025X075
- C6: value 4µ7 -> 47n; device rcl:CPOL-EUE2-5 -> rcl:C-EU050-025X075
- C7, C8: value 100n -> 47n; device rcl:C-EUC1206 -> rcl:C-EU050-025X075
- IC1: value 78L05 -> MEGA48-P; device v-reg:78XXL -> atmel:MEGA8-P
- R1: value 1k -> 10K; device rcl:R-EU_R1206 -> rcl:R-EU_0207/10
- R10, R2, R3, R5, R6, R7, R9: device rcl:R-EU_R1206 -> rcl:R-EU_0207/10
- R4: value 10R -> 1k; device rcl:R-EU_0414/15 -> rcl:R-EU_0207/10
- R8: value (none) -> 1k; device rcl:R-EU_R1206 -> rcl:R-EU_0207/10
Connections:
- removed net !CE: H1.!CE, IC2A.B4
- removed net !RD: H1.!RD, IC2A.B1, IC3A.DIR
- removed net !RST: H1.!RST, IC2A.B3
- removed net !WR: H1.!WR, IC2A.B2
- removed net +12V: C12.+, C6.+, C7.1, IC1.IN, Q2.S, Q5.S, X1-2.KL
- removed net +24V: C10.+, C11.+, C5.+, Q7.S, Q9.S, X1-3.KL
- removed net +5V: C1.1, C2.1, C3.1, C4.1, C8.1, C9.+, H1.VCC, IC1.OUT, IC2A.DIR, IC2P.VCC, IC3P.VCC, SJ1.1, SJ2.1, X3PWR.5V@1, X3PWR.5V@2
- removed net A0: H1.A0, IC2A.B6
- removed net A1: H1.A1, IC2A.B7
- removed net A2: H1.A2, IC2A.B8
- removed net BL: H1.BL_DISP, JP2.3, R4.2
- removed net BUZZ: H1.GND_BUZZ, Q3.D
- removed net C/D: H1.C/D, IC2A.B5
- removed net D0: H1.D0, IC3A.B1
- removed net D1: H1.D1, IC3A.B2
- removed net D2: H1.D2, IC3A.B3
- removed net D3: H1.D3, IC3A.B4
- removed net D4: H1.D4, IC3A.B5
- removed net D5: H1.D5, IC3A.B6
- removed net D6: H1.D6, IC3A.B7
- removed net D7: H1.D7, IC3A.B8
- removed net ENC_A: X2-1.S, X3PORTB.PB4
- removed net ENC_B: X2-3.S, X3PORTB.PB5
- removed net ENC_UB: X3PORTB.PB7, X5-1.S
- removed net FS1: R1.1
- removed net IN_!CE: IC2A.A4, X3PORTB.PB14
- removed net IN_!RD: IC2A.A1, X3PORTB.PB11
- removed net IN_!RST: IC2A.A3, X3PORTB.PB13
- removed net IN_!WR: IC2A.A2, X3PORTB.PB12
- removed net IN_A0: IC2A.A6, X3PORTB.PB0
- removed net IN_A1: IC2A.A7, X3PORTB.PB1
- removed net IN_A2: IC2A.A8, X3PORTB.PB2
- removed net IN_BL: R5.1, X3PORTA.PA1
- removed net IN_BUZZ: R6.1, X3PORTA.PA2
- removed net IN_C/D: IC2A.A5, X3PORTB.PB15
- removed net IN_D0: IC3A.A1, X3PORTE.PE8
- removed net IN_D1: IC3A.A2, X3PORTE.PE9
- removed net IN_D2: IC3A.A3, X3PORTE.PE10
- removed net IN_D3: IC3A.A4, X3PORTE.PE11
- removed net IN_D4: IC3A.A5, X3PORTE.PE12
- removed net IN_D5: IC3A.A6, X3PORTE.PE13
- removed net IN_D6: IC3A.A7, X3PORTE.PE14
- removed net IN_D7: IC3A.A8, X3PORTE.PE15
- removed net IN_LED: R8.1, X3PORTA.PA3
- removed net IN_OUT1: R12.1, X3PORTA.PA4
- removed net IN_OUT2: R10.1, X3PORTA.PA8
- removed net LED: H1.BL_LED, Q5.D
- removed net LED1: Q7.D, X6-2.KL
- removed net LED2: Q9.D, X4-2.KL
- removed net MD2: R2.1
- removed net N$1: R1.2, SJ1.2
- removed net N$10: Q7.G, R9.2
- removed net N$11: Q4.G, R8.2
- removed net N$12: Q6.D, R9.1
- removed net N$13: Q6.G, R10.2
- removed net N$14: Q9.G, R11.2
- removed net N$15: Q8.D, R11.1
- removed net N$16: Q8.G, R12.2
- removed net N$20: X10-2.S, X3PORTD.PD8
- removed net N$21: X10-1.S, X3PORTD.PD9
- removed net N$22: X3PORTD.PD10, X9-2.S
- removed net N$23: X3PORTD.PD11, X9-1.S
- removed net N$24: X3PORTD.PD12, X8-2.S
- removed net N$25: X3PORTD.PD13, X8-1.S
- removed net N$26: X3PORTD.PD14, X7-2.S
- removed net N$27: X3PORTD.PD15, X7-1.S
- removed net N$7: Q5.G, R7.2
- removed net N$8: Q3.G, R6.2
- removed net N$9: Q4.D, R7.1
- removed net VBAT: H1.VBAT
- new net KEY0: R6.2
- new net KEY1: R7.2
- new net KEY2: R8.2
- new net KEY3: R9.2
- new net MISO: IC1.PB4(MISO), JP1.1
- new net MOSI: IC1.PB3(MOSI/OC2), JP1.4
- new net OUT1: IC1.PC0(ADC0), R2.1
- new net OUT2: IC1.PC1(ADC1), R3.1
- new net OUT3: IC1.PC2(ADC2), R4.1
- new net OUT4: IC1.PC3(ADC3), R5.1
- new net RESET: IC1.PC6(/RESET), JP1.5, R1.1
- new net SCK: IC1.PB5(SCK), JP1.3
- new net SNS0: C5.1, IC1.PD0(RXD)
- new net SNS1: C6.1, IC1.PD2(INT0)
- new net SNS2: C7.1, IC1.PD4(XCK/T0)
- new net SNS3: C8.1, IC1.PD6(AIN0)
- new net SNSK0: C5.2, IC1.PD1(TXD), R6.1
- new net SNSK1: C6.2, IC1.PD3(INT1), R7.1
- new net SNSK2: C7.2, IC1.PD5(T1), R8.1
- new net SNSK3: C8.2, IC1.PD7(AIN1), R9.1
- new net VCC: C1.1, C4.+, IC1.AVCC, IC1.VCC@1, J1-2.S, R1.2, R10.2
- net GND: now also C4.-, IC1.GND@1, J1-1.S, JP1.6, LED1.C; no longer C10.-, C11.-, C12.-, C2.2, C3.2, C4.2, C5.-, C6.-, C7.2, C8.2, C9.-, H1.GND, IC2A.G, IC2P.GND, IC3A.G, IC3P.GND, JP2.1, Q1.S, Q3.S, Q4.S, Q6.S, Q8.S, SJ1.3, SJ2.3, X1-1.KL, X10-3.S, X2-2.S, X3PWR.GND@1, X3PWR.GND@10, X3PWR.GND@2, X3PWR.GND@3, X3PWR.GND@4, X3PWR.GND@5, X3PWR.GND@6, X3PWR.GND@7, X3PWR.GND@8, X3PWR.GND@9, X4-1.KL, X5-2.S, X6-1.KL, X7-3.S, X8-3.S, X9-3.S
- net N$2: now also J2-4.S; no longer SJ2.2
- net N$3: now also J2-3.S; no longer Q2.G
- net N$4: now also J2-2.S, R4.2; no longer Q1.D, R3.1
- net N$5: now also J2-1.S, R5.2; no longer Q2.D, R4.1
- net N$6: now also LED1.A, R10.1; no longer Q1.G, R5.2
Other:
- moved on the sheet: C1, C7, C8, R1, R10, R2, R3, R4, R5, R6, R7, R8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
